Commit message: Improve collision guard and lidar placement

File: src/mrt_description/urdf/gazebo_plugins.xacro (robot description, xacro)
@@ -6,10 +6,16 @@
     </gazebo>
     <gazebo reference="left_wheel_link">
-      <mu1>1.0</mu1>
-      <mu2>1.0</mu2>
+      <mu1>1.5</mu1>
+      <mu2>1.5</mu2>
+      <slip1>0.02</slip1>
+      <slip2>0.0</slip2>
+      <fdir1>0 0 1</fdir1>
     </gazebo>
     <gazebo reference="right_wheel_link">
-      <mu1>1.0</mu1>
-      <mu2>1.0</mu2>
+      <mu1>1.5</mu1>
+      <mu2>1.5</mu2>
+      <slip1>0.02</slip1>
+      <slip2>0.0</slip2>
+      <fdir1>0 0 1</fdir1>
     </gazebo>
     <gazebo reference="front_caster_link">
@@ -29,10 +35,28 @@
         <wheel_separation>0.51</wheel_separation>
         <wheel_radius>0.08</wheel_radius>
+        <max_linear_velocity>0.45</max_linear_velocity>
+        <min_linear_velocity>-0.35</min_linear_velocity>
+        <max_angular_velocity>1.2</max_angular_velocity>
+        <min_angular_velocity>-1.2</min_angular_velocity>
+        <max_linear_acceleration>0.8</max_linear_acceleration>
+        <min_linear_acceleration>-1.2</min_linear_acceleration>
+        <max_angular_acceleration>2.0</max_angular_acceleration>
+        <min_angular_acceleration>-2.0</min_angular_acceleration>
+        <max_linear_jerk>6.0</max_linear_jerk>
+        <min_linear_jerk>-6.0</min_linear_jerk>
+        <max_angular_jerk>8.0</max_angular_jerk>
+        <min_angular_jerk>-8.0</min_angular_jerk>
         <odom_publish_frequency>50</odom_publish_frequency>
-        <topic>${robot_name}/cmd_vel</topic>
+        <topic>${robot_name}/cmd_vel_safe</topic>
         <odom_topic>${robot_name}/odom</odom_topic>
         <tf_topic>${robot_name}/tf</tf_topic>
         <frame_id>${robot_name}/odom</frame_id>
         <child_frame_id>${robot_name}/base_footprint</child_frame_id>
+      </plugin>
+      <plugin
+        filename="gz-sim-joint-state-publisher-system"
+        name="gz::sim::systems::JointStatePublisher">
+        <joint_name>left_wheel_joint</joint_name>
+        <joint_name>right_wheel_joint</joint_name>
       </plugin>
     </gazebo>

File: src/mrt_description/urdf/robot.urdf.xacro (robot description, xacro)
@@ -8,4 +8,7 @@
   <xacro:arg name="camera_enabled" default="true"/>
   <xacro:arg name="use_gazebo_plugins" default="false"/>
+  <xacro:arg name="lidar_x" default="0.22"/>
+  <xacro:arg name="lidar_y" default="0"/>
+  <xacro:arg name="lidar_z" default="0.045"/>
   <xacro:include filename="$(find mrt_description)/urdf/materials.xacro"/>
   <xacro:include filename="$(find mrt_description)/urdf/inertials.xacro"/>
@@ -17,5 +20,5 @@
   <xacro:mrt_base robot_color="$(arg robot_color)"/>
   <xacro:mrt_wheels/>
-  <xacro:mrt_lidar/>
+  <xacro:mrt_lidar x="$(arg lidar_x)" y="$(arg lidar_y)" z="$(arg lidar_z)"/>
   <xacro:mrt_imu/>
   <xacro:mrt_camera enabled="$(arg camera_enabled)"/>

File: src/mrt_description/urdf/sensors.xacro (robot description, xacro)
@@ -1,5 +1,5 @@
 <?xml version="1.0"?>
 <robot xmlns:xacro="http://www.ros.org/wiki/xacro">
-  <xacro:macro name="mrt_lidar">
+  <xacro:macro name="mrt_lidar" params="x:=0.22 y:=0 z:=0.045">
     <link name="lidar_link">
       <visual>
@@ -21,5 +21,5 @@
       <parent link="top_deck_link"/>
       <child link="lidar_link"/>
-      <origin xyz="0.22 0 0.045" rpy="0 0 0"/>
+      <origin xyz="${x} ${y} ${z}" rpy="0 0 0"/>
     </joint>
   </xacro:macro>
