Commit message: feat: add predictive dynamic navigation lab

File: src/predictive_nav_description/urdf/base.xacro (robot description, xacro)
@@ -1,26 +1,29 @@
 <?xml version="1.0"?>
 <robot xmlns:xacro="http://www.ros.org/wiki/xacro">
-  <xacro:macro name="predictive_nav_base" params="robot_color:=predictive_nav_blue">
+  <xacro:macro name="predictive_nav_base" params="robot_color:=predictive_nav_blue base_radius:=0.110 base_height:=0.060 base_ground_clearance:=0.005 base_link_z:=0.0325">
     <link name="base_footprint"/>
     <joint name="base_footprint_joint" type="fixed">
       <parent link="base_footprint"/>
       <child link="base_link"/>
-      <origin xyz="0 0 0.095" rpy="0 0 0"/>
+      <!-- base_footprint is the ground-plane centre; base_link is the wheel axle plane. -->
+      <origin xyz="0 0 ${base_link_z}" rpy="0 0 0"/>
     </joint>
     <link name="base_link">
       <visual>
-        <origin xyz="0 0 0.02" rpy="0 0 0"/>
+        <origin xyz="0 0 ${base_ground_clearance + base_height / 2.0 - base_link_z}" rpy="0 0 0"/>
         <geometry>
-          <box size="0.62 0.46 0.18"/>
+          <cylinder radius="${base_radius}" length="${base_height}"/>
         </geometry>
         <material name="${robot_color}"/>
       </visual>
       <collision>
-        <origin xyz="0 0 0.02" rpy="0 0 0"/>
+        <origin xyz="0 0 ${base_ground_clearance + base_height / 2.0 - base_link_z}" rpy="0 0 0"/>
         <geometry>
-          <box size="0.62 0.46 0.18"/>
+          <!-- Simple circular collision body: appropriate for Nav2/Gazebo, not a CAD model. -->
+          <cylinder radius="${base_radius}" length="${base_height}"/>
         </geometry>
       </collision>
-      <xacro:predictive_nav_box_inertia mass="16.0" x="0.62" y="0.46" z="0.18"/>
+      <!-- PROVISIONAL_DESIGN_VALUE: update mass/inertia after the robot is weighed. -->
+      <xacro:predictive_nav_cylinder_inertia_z mass="4.0" radius="${base_radius}" length="${base_height}"/>
     </link>
     <link name="top_deck_link">
@@ -28,62 +31,15 @@
         <origin xyz="0 0 0" rpy="0 0 0"/>
         <geometry>
-          <box size="0.56 0.40 0.035"/>
+          <cylinder radius="${base_radius - 0.006}" length="0.004"/>
         </geometry>
         <material name="predictive_nav_dark_grey"/>
       </visual>
-      <collision>
-        <origin xyz="0 0 0" rpy="0 0 0"/>
-        <geometry>
-          <box size="0.56 0.40 0.035"/>
-        </geometry>
-      </collision>
-      <xacro:predictive_nav_box_inertia mass="1.0" x="0.56" y="0.40" z="0.035"/>
+      <!-- Deck/electronics are visual-only so they do not enlarge collision or Nav2 footprint. -->
+      <xacro:predictive_nav_cylinder_inertia_z mass="0.15" radius="${base_radius - 0.006}" length="0.004"/>
     </link>
     <joint name="top_deck_joint" type="fixed">
       <parent link="base_link"/>
       <child link="top_deck_link"/>
-      <origin xyz="0 0 0.128" rpy="0 0 0"/>
-    </joint>
-    <link name="front_bumper_link">
-      <visual>
-        <origin xyz="0 0 0" rpy="0 0 0"/>
-        <geometry>
-          <box size="0.04 0.44 0.09"/>
-        </geometry>
-        <material name="predictive_nav_dark_grey"/>
-      </visual>
-      <collision>
-        <origin xyz="0 0 0" rpy="0 0 0"/>
-        <geometry>
-          <box size="0.04 0.44 0.09"/>
-        </geometry>
-      </collision>
-      <xacro:predictive_nav_box_inertia mass="0.8" x="0.04" y="0.44" z="0.09"/>
-    </link>
-    <joint name="front_bumper_joint" type="fixed">
-      <parent link="base_link"/>
-      <child link="front_bumper_link"/>
-      <origin xyz="0.335 0 0.02" rpy="0 0 0"/>
-    </joint>
-    <link name="rear_bumper_link">
-      <visual>
-        <origin xyz="0 0 0" rpy="0 0 0"/>
-        <geometry>
-          <box size="0.035 0.42 0.08"/>
-        </geometry>
-        <material name="predictive_nav_dark_grey"/>
-      </visual>
-      <collision>
-        <origin xyz="0 0 0" rpy="0 0 0"/>
-        <geometry>
-          <box size="0.035 0.42 0.08"/>
-        </geometry>
-      </collision>
-      <xacro:predictive_nav_box_inertia mass="0.6" x="0.035" y="0.42" z="0.08"/>
-    </link>
-    <joint name="rear_bumper_joint" type="fixed">
-      <parent link="base_link"/>
-      <child link="rear_bumper_link"/>
-      <origin xyz="-0.335 0 0.02" rpy="0 0 0"/>
+      <origin xyz="0 0 ${base_ground_clearance + base_height - base_link_z}" rpy="0 0 0"/>
     </joint>
   </xacro:macro>

File: src/predictive_nav_description/urdf/gazebo_plugins.xacro (robot description, xacro)
@@ -1,5 +1,5 @@
 <?xml version="1.0"?>
 <robot xmlns:xacro="http://www.ros.org/wiki/xacro">
-  <xacro:macro name="predictive_nav_gazebo_plugins" params="topic_prefix:=nav_robot odom_frame:=odom base_frame:=base_footprint">
+  <xacro:macro name="predictive_nav_gazebo_plugins" params="topic_prefix:=nav_robot odom_frame:=odom base_frame:=base_footprint wheel_separation:=0.220 wheel_radius:=0.0325">
     <gazebo reference="base_link">
       <material>Gazebo/Blue</material>
@@ -26,6 +26,7 @@
         <left_joint>left_wheel_joint</left_joint>
         <right_joint>right_wheel_joint</right_joint>
-        <wheel_separation>0.51</wheel_separation>
-        <wheel_radius>0.08</wheel_radius>
+        <!-- Passed from robot.urdf.xacro: one source for link geometry and DiffDrive kinematics. -->
+        <wheel_separation>${wheel_separation}</wheel_separation>
+        <wheel_radius>${wheel_radius}</wheel_radius>
         <max_linear_velocity>0.45</max_linear_velocity>
         <min_linear_velocity>-0.35</min_linear_velocity>

File: src/predictive_nav_description/urdf/robot.urdf.xacro (robot description, xacro)
@@ -4,7 +4,43 @@
   <xacro:arg name="robot_color" default="predictive_nav_blue"/>
   <xacro:arg name="use_gazebo_plugins" default="false"/>
-  <xacro:arg name="lidar_x" default="0.22"/>
-  <xacro:arg name="lidar_y" default="0"/>
-  <xacro:arg name="lidar_z" default="0.045"/>
+  <!--
+    Real-robot geometry register
+    ============================
+    Hardware-specification values:
+      base_radius=0.110 m       (220 mm circular aluminium chassis)
+      wheel_radius=0.0325 m     (65 mm nominal drive-wheel diameter)
+    Values marked PROVISIONAL_DESIGN_VALUE make the simulation runnable;
+    they are not measurements of the unfinished robot.  Replace every
+    REAL_ROBOT_CALIBRATION item after the mechanical assembly is complete.
+    Keep Nav2's robot_radius and a future DynamicRiskCritic robot_radius_m
+    equal to the final *maximum mechanical radius plus their chosen safety
+    margin*.  See predictive_nav_bringup/config/nav2_dwb.yaml.
+  -->
+  <xacro:arg name="base_radius" default="0.110"/>
+  <xacro:arg name="base_height" default="0.060"/> <!-- PROVISIONAL_DESIGN_VALUE -->
+  <xacro:arg name="base_ground_clearance" default="0.005"/> <!-- PROVISIONAL_DESIGN_VALUE -->
+  <xacro:arg name="wheel_radius" default="0.0325"/>
+  <xacro:arg name="wheel_width" default="0.027"/> <!-- REAL_ROBOT_CALIBRATION; provisional design value -->
+  <xacro:arg name="wheel_separation" default="0.220"/> <!-- REAL_ROBOT_CALIBRATION; provisional design value -->
+  <xacro:arg name="wheel_x" default="0.0"/> <!-- REAL_ROBOT_CALIBRATION; provisional design value -->
+  <xacro:arg name="caster_ball_radius" default="0.015"/> <!-- REAL_ROBOT_CALIBRATION; provisional design value -->
+  <xacro:arg name="caster_1_x" default="0.065"/> <!-- REAL_ROBOT_CALIBRATION; provisional design value -->
+  <xacro:arg name="caster_1_y" default="0.0"/> <!-- REAL_ROBOT_CALIBRATION; provisional design value -->
+  <xacro:arg name="caster_2_x" default="-0.065"/> <!-- REAL_ROBOT_CALIBRATION; provisional design value -->
+  <xacro:arg name="caster_2_y" default="0.0"/> <!-- REAL_ROBOT_CALIBRATION; provisional design value -->
+  <xacro:arg name="lidar_x" default="0.0"/> <!-- REAL_ROBOT_CALIBRATION; relative to base_link -->
+  <xacro:arg name="lidar_y" default="0.0"/> <!-- REAL_ROBOT_CALIBRATION; provisional design value -->
+  <!-- Center of the simple 55 mm-high LiDAR visual: its bottom rests on the deck. -->
+  <xacro:arg name="lidar_z" default="0.060"/> <!-- REAL_ROBOT_CALIBRATION; provisional design value -->
+  <xacro:arg name="lidar_roll" default="0.0"/> <!-- REAL_ROBOT_CALIBRATION -->
+  <xacro:arg name="lidar_pitch" default="0.0"/> <!-- REAL_ROBOT_CALIBRATION -->
+  <xacro:arg name="lidar_yaw" default="0.0"/> <!-- REAL_ROBOT_CALIBRATION -->
+  <xacro:arg name="imu_x" default="0.0"/> <!-- REAL_ROBOT_CALIBRATION; relative to base_link -->
+  <xacro:arg name="imu_y" default="0.0"/> <!-- REAL_ROBOT_CALIBRATION; provisional design value -->
+  <!-- Placeholder IMU visual also rests on the deck; final IMU pose is TBD. -->
+  <xacro:arg name="imu_z" default="0.045"/> <!-- REAL_ROBOT_CALIBRATION; provisional design value -->
+  <xacro:arg name="imu_roll" default="0.0"/> <!-- REAL_ROBOT_CALIBRATION -->
+  <xacro:arg name="imu_pitch" default="0.0"/> <!-- REAL_ROBOT_CALIBRATION -->
+  <xacro:arg name="imu_yaw" default="0.0"/> <!-- REAL_ROBOT_CALIBRATION -->
   <xacro:include filename="$(find predictive_nav_description)/urdf/materials.xacro"/>
   <xacro:include filename="$(find predictive_nav_description)/urdf/inertials.xacro"/>
@@ -13,10 +49,29 @@
   <xacro:include filename="$(find predictive_nav_description)/urdf/sensors.xacro"/>
   <xacro:include filename="$(find predictive_nav_description)/urdf/gazebo_plugins.xacro"/>
-  <xacro:predictive_nav_base robot_color="$(arg robot_color)"/>
-  <xacro:predictive_nav_wheels/>
-  <xacro:predictive_nav_lidar x="$(arg lidar_x)" y="$(arg lidar_y)" z="$(arg lidar_z)"/>
-  <xacro:predictive_nav_imu/>
+  <xacro:predictive_nav_base
+    robot_color="$(arg robot_color)"
+    base_radius="$(arg base_radius)"
+    base_height="$(arg base_height)"
+    base_ground_clearance="$(arg base_ground_clearance)"
+    base_link_z="$(arg wheel_radius)"/>
+  <xacro:predictive_nav_wheels
+    wheel_radius="$(arg wheel_radius)"
+    wheel_width="$(arg wheel_width)"
+    wheel_separation="$(arg wheel_separation)"
+    wheel_x="$(arg wheel_x)"
+    caster_ball_radius="$(arg caster_ball_radius)"
+    caster_1_x="$(arg caster_1_x)" caster_1_y="$(arg caster_1_y)"
+    caster_2_x="$(arg caster_2_x)" caster_2_y="$(arg caster_2_y)"/>
+  <xacro:predictive_nav_lidar
+    x="$(arg lidar_x)" y="$(arg lidar_y)" z="$(arg lidar_z)"
+    roll="$(arg lidar_roll)" pitch="$(arg lidar_pitch)" yaw="$(arg lidar_yaw)"/>
+  <xacro:predictive_nav_imu
+    x="$(arg imu_x)" y="$(arg imu_y)" z="$(arg imu_z)"
+    roll="$(arg imu_roll)" pitch="$(arg imu_pitch)" yaw="$(arg imu_yaw)"/>
   <xacro:if value="$(arg use_gazebo_plugins)">
-    <xacro:predictive_nav_gazebo_plugins topic_prefix="$(arg robot_name)"/>
+    <xacro:predictive_nav_gazebo_plugins
+      topic_prefix="$(arg robot_name)"
+      wheel_separation="$(arg wheel_separation)"
+      wheel_radius="$(arg wheel_radius)"/>
   </xacro:if>
 </robot>

File: src/predictive_nav_description/urdf/sensors.xacro (robot description, xacro)
@@ -1,5 +1,5 @@
 <?xml version="1.0"?>
 <robot xmlns:xacro="http://www.ros.org/wiki/xacro">
-  <xacro:macro name="predictive_nav_lidar" params="x:=0.22 y:=0 z:=0.045">
+  <xacro:macro name="predictive_nav_lidar" params="x:=0.0 y:=0.0 z:=0.060 roll:=0.0 pitch:=0.0 yaw:=0.0">
     <link name="lidar_link">
       <visual>
@@ -19,10 +19,11 @@
     </link>
     <joint name="lidar_joint" type="fixed">
-      <parent link="top_deck_link"/>
+      <!-- Pose is explicitly relative to base_link for later survey/calibration. -->
+      <parent link="base_link"/>
       <child link="lidar_link"/>
-      <origin xyz="${x} ${y} ${z}" rpy="0 0 0"/>
+      <origin xyz="${x} ${y} ${z}" rpy="${roll} ${pitch} ${yaw}"/>
     </joint>
   </xacro:macro>
-  <xacro:macro name="predictive_nav_imu">
+  <xacro:macro name="predictive_nav_imu" params="x:=0.0 y:=0.0 z:=0.045 roll:=0.0 pitch:=0.0 yaw:=0.0">
     <link name="imu_link">
       <visual>
@@ -33,10 +34,5 @@
         <material name="predictive_nav_black"/>
       </visual>
-      <collision>
-        <origin xyz="0 0 0" rpy="0 0 0"/>
-        <geometry>
-          <box size="0.05 0.04 0.02"/>
-        </geometry>
-      </collision>
+      <!-- Placeholder only: no IMU model/driver is implied and it has no collision. -->
       <xacro:predictive_nav_box_inertia mass="0.08" x="0.05" y="0.04" z="0.02"/>
     </link>
@@ -44,5 +40,5 @@
       <parent link="base_link"/>
       <child link="imu_link"/>
-      <origin xyz="0 0 0.125" rpy="0 0 0"/>
+      <origin xyz="${x} ${y} ${z}" rpy="${roll} ${pitch} ${yaw}"/>
     </joint>
   </xacro:macro>

File: src/predictive_nav_description/urdf/wheels.xacro (robot description, xacro)
@@ -1,10 +1,10 @@
 <?xml version="1.0"?>
 <robot xmlns:xacro="http://www.ros.org/wiki/xacro">
-  <xacro:macro name="predictive_nav_wheels">
+  <xacro:macro name="predictive_nav_wheels" params="wheel_radius:=0.0325 wheel_width:=0.027 wheel_separation:=0.220 wheel_x:=0.0 caster_ball_radius:=0.015 caster_1_x:=0.065 caster_1_y:=0.0 caster_2_x:=-0.065 caster_2_y:=0.0">
     <link name="left_wheel_link">
       <visual>
         <origin xyz="0 0 0" rpy="1.57079632679 0 0"/>
         <geometry>
-          <cylinder radius="0.08" length="0.045"/>
+          <cylinder radius="${wheel_radius}" length="${wheel_width}"/>
         </geometry>
         <material name="predictive_nav_black"/>
@@ -13,13 +13,14 @@
         <origin xyz="0 0 0" rpy="1.57079632679 0 0"/>
         <geometry>
-          <cylinder radius="0.08" length="0.045"/>
+          <cylinder radius="${wheel_radius}" length="${wheel_width}"/>
         </geometry>
       </collision>
-      <xacro:predictive_nav_cylinder_inertia_x mass="0.75" radius="0.08" length="0.045"/>
+      <xacro:predictive_nav_cylinder_inertia_x mass="0.18" radius="${wheel_radius}" length="${wheel_width}"/>
     </link>
     <joint name="left_wheel_joint" type="continuous">
       <parent link="base_link"/>
       <child link="left_wheel_link"/>
-      <origin xyz="0 0.255 -0.015" rpy="0 0 0"/>
+      <origin xyz="${wheel_x} ${wheel_separation / 2.0} 0" rpy="0 0 0"/>
+      <!-- ROS convention: +Y wheel axle, +X forward. -->
       <axis xyz="0 1 0"/>
     </joint>
@@ -28,5 +29,5 @@
         <origin xyz="0 0 0" rpy="1.57079632679 0 0"/>
         <geometry>
-          <cylinder radius="0.08" length="0.045"/>
+          <cylinder radius="${wheel_radius}" length="${wheel_width}"/>
         </geometry>
         <material name="predictive_nav_black"/>
@@ -35,20 +36,21 @@
         <origin xyz="0 0 0" rpy="1.57079632679 0 0"/>
         <geometry>
-          <cylinder radius="0.08" length="0.045"/>
+          <cylinder radius="${wheel_radius}" length="${wheel_width}"/>
         </geometry>
       </collision>
-      <xacro:predictive_nav_cylinder_inertia_x mass="0.75" radius="0.08" length="0.045"/>
+      <xacro:predictive_nav_cylinder_inertia_x mass="0.18" radius="${wheel_radius}" length="${wheel_width}"/>
     </link>
     <joint name="right_wheel_joint" type="continuous">
       <parent link="base_link"/>
       <child link="right_wheel_link"/>
-      <origin xyz="0 -0.255 -0.015" rpy="0 0 0"/>
+      <origin xyz="${wheel_x} ${-wheel_separation / 2.0} 0" rpy="0 0 0"/>
       <axis xyz="0 1 0"/>
     </joint>
+    <!-- Two passive ball casters.  Their size and mounting points are calibration items. -->
     <link name="front_caster_link">
       <visual>
         <origin xyz="0 0 0" rpy="0 0 0"/>
         <geometry>
-          <sphere radius="0.035"/>
+          <sphere radius="${caster_ball_radius}"/>
         </geometry>
         <material name="predictive_nav_light_grey"/>
@@ -57,13 +59,13 @@
         <origin xyz="0 0 0" rpy="0 0 0"/>
         <geometry>
-          <sphere radius="0.035"/>
+          <sphere radius="${caster_ball_radius}"/>
         </geometry>
       </collision>
-      <xacro:predictive_nav_cylinder_inertia_z mass="0.2" radius="0.035" length="0.035"/>
+      <xacro:predictive_nav_cylinder_inertia_z mass="0.05" radius="${caster_ball_radius}" length="${caster_ball_radius * 2.0}"/>
     </link>
     <joint name="front_caster_joint" type="fixed">
       <parent link="base_link"/>
       <child link="front_caster_link"/>
-      <origin xyz="0.24 0 -0.06" rpy="0 0 0"/>
+      <origin xyz="${caster_1_x} ${caster_1_y} ${caster_ball_radius - wheel_radius}" rpy="0 0 0"/>
     </joint>
     <link name="rear_caster_link">
@@ -71,5 +73,5 @@
         <origin xyz="0 0 0" rpy="0 0 0"/>
         <geometry>
-          <sphere radius="0.035"/>
+          <sphere radius="${caster_ball_radius}"/>
         </geometry>
         <material name="predictive_nav_light_grey"/>
@@ -78,13 +80,13 @@
         <origin xyz="0 0 0" rpy="0 0 0"/>
         <geometry>
-          <sphere radius="0.035"/>
+          <sphere radius="${caster_ball_radius}"/>
         </geometry>
       </collision>
-      <xacro:predictive_nav_cylinder_inertia_z mass="0.2" radius="0.035" length="0.035"/>
+      <xacro:predictive_nav_cylinder_inertia_z mass="0.05" radius="${caster_ball_radius}" length="${caster_ball_radius * 2.0}"/>
     </link>
     <joint name="rear_caster_joint" type="fixed">
       <parent link="base_link"/>
       <child link="rear_caster_link"/>
-      <origin xyz="-0.24 0 -0.06" rpy="0 0 0"/>
+      <origin xyz="${caster_2_x} ${caster_2_y} ${caster_ball_radius - wheel_radius}" rpy="0 0 0"/>
     </joint>
   </xacro:macro>
